File: ESP32-C3_ePaper/ESP32-C3_ePaper/ESP32-C3_ePaper.kicad_sch (KiCad schematic)
At the start: 3 parts, among them J1 e-Paper, U1 ESP32-C3 SuperMini

Commit message: .
Parts:
- removed U2: ~, symbol Alexander Symbols Library:ESP32C3_ZenBoard
- added U3: ~, symbol ProjectLibrary:ESP32C3_ZenBoard
Connections:
- net +3V3: now also U3.1 (3V3)
- net BUSY: now also U3.15 (GPIO3)
- net CLK: now also U3.12 (Tx)
- net CS: now also U3.6 (GPIO7)
- net DC: now also U3.17 (GPIO1)
- net DIN: now also U3.5 (GPIO6)
- net GNDD: now also U3.9 (G)
- net RST: now also U3.16 (GPIO2)
Changed lines of the file:
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@@
+	)
+	(symbol
+		(lib_id "ProjectLibrary:ESP32C3_ZenBoard")
+		(at 83.82 105.41 0)
+		(unit 1)
+		(exclude_from_sim no)
+		(in_bom yes)
+		(on_board yes)
+		(dnp no)
+		(fields_autoplaced yes)
+		(property "Reference" "U3"
+			(at 84.455 104.14 0)
+			(effects
+				(font
+					(size 1.27 1.27)
+				)
+			)
+		)
+		(property "Value" "~"
+			(at 84.455 106.68 0)
+			(effects
+				(font
+					(size 1.27 1.27)
+				)
+			)
+		)
+		(property "Footprint" ""
+			(at 83.82 105.41 0)
+			(effects
+				(font
+					(size 1.27 1.27)
+				)
+				(hide yes)
+			)
+		)
+		(property "Datasheet" ""
+			(at 83.82 105.41 0)
+			(effects
+				(font
+					(size 1.27 1.27)
+				)
+				(hide yes)
+			)
+		)
+		(property "Description" ""
+			(at 83.82 105.41 0)
+			(effects
+				(font
+					(size 1.27 1.27)
+				)
+				(hide yes)
+			)
+		)
+		(pin "8"
+		)
+		(pin "9"
+		)
+		(pin "7"
+		)
+		(pin "12"
+		)
+		(pin "18"
+		)
+		(pin "16"
+		)
+		(pin "13"
+		)
+		(pin "15"
+		)
+		(pin "17"
+		)
+		(pin "10"
+		)
+		(pin "1"
+		)
+		(pin "4"
+		)
+		(pin "5"
+		)
+		(pin "2"
+		)
+		(pin "11"
+		)
+		(pin "6"
+		)
+		(pin "3"
+		)
+		(pin "14"
+		)
+		(instances
+			(project ""
+				(path "/95feff10-2965-4a71-88b6-e41b0fca8232"
+					(reference "U3")
+					(unit 1)
+				)
+			)
+		)
 	)
 	(symbol
@@
 					(unit 1)
 				)
-			)
-		)
-	)
-	(symbol
-		(lib_id "Alexander Symbols Library:ESP32C3_ZenBoard")
-		(at 83.82 105.41 0)
-		(unit 1)
-		(exclude_from_sim no)
-		(in_bom yes)
-		(on_board yes)
-		(dnp no)
-		(fields_autoplaced yes)
-		(property "Reference" "U2"
-			(at 84.455 104.14 0)
-			(effects
-				(font
-					(size 1.27 1.27)
-				)
-			)
-		)
-		(property "Value" "~"
-			(at 84.455 106.68 0)
-			(effects
-				(font
-					(size 1.27 1.27)
-				)
-			)
-		)
-		(property "Footprint" ""
-			(at 83.82 105.41 0)
-			(effects
-				(font
-					(size 1.27 1.27)
-				)
-				(hide yes)
-			)
-		)
-		(property "Datasheet" ""
-			(at 83.82 105.41 0)
-			(effects
-				(font
-					(size 1.27 1.27)
-				)
-				(hide yes)
-			)
-		)
-		(property "Description" ""
-			(at 83.82 105.41 0)
-			(effects
-				(font
-					(size 1.27 1.27)
-				)
-				(hide yes)
-			)
-		)
-		(pin "2"
-		)
-		(pin "12"
-		)
-		(pin "11"
-		)
-		(pin "13"
-		)
-		(pin "18"
-		)
-		(pin "10"
-		)
-		(pin "9"
-		)
-		(pin "8"
-		)
-		(pin "7"
-		)
-		(pin "6"
-		)
-		(pin "5"
-		)
-		(pin "4"
-		)
-		(pin "3"
-		)
-		(pin "15"
-		)
-		(pin "1"
-		)
-		(pin "16"
-		)
-		(pin "17"
-		)
-		(pin "14"
-		)
-		(instances
-			(project ""
-				(path "/95feff10-2965-4a71-88b6-e41b0fca8232"
-					(reference "U2")
-					(unit 1)
-				)
